Commit message: Added friction parameter

File: robot/description/roller/roller.urdf.xacro (robot description, xacro)
@@ -9,5 +9,8 @@
 	  <child link="${prefix}_roller_link"/>
 	  <xacro:insert_block name="joint_axis"/>
-    <dynamics damping="0.0" friction="1.0"/>
+    <!--
+      Setting friction too high (1.0 tested) result in weird movement and behavior
+    -->
+    <dynamics damping="0.0" friction="0.01"/>
 	</joint>
 	<link name="${prefix}_roller_link">
@@ -42,5 +45,5 @@
             <ode>
                 <max_vel>10</max_vel>
-                <min_depth>0.001</min_depth>
+                <min_depth>0.01</min_depth>
             </ode>
             </contact>
