Commit message: Changed params

File: robot/description/ros2_control.xacro (robot description, xacro)
@@ -4,14 +4,17 @@
         <hardware>
             <plugin>omnidrive3_rppico/omnidrive3RpPicoHardware</plugin>
-            <param name="wheel1_name">roue_avant_joint</param>
-            <param name="wheel2_name">roue_gauche_joint</param>
-            <param name="wheel3_name">roue_arriere_joint</param>
+            <!--
+            <param name="device">/dev/pts/6</param>
+            -->
+            <param name="device">/dev/pts/69</param>
+            <param name="baudrate">115200</param>
+            <param name="wheel1_name">first_wheel_joint</param>
+            <param name="wheel2_name">second_wheel_joint</param>
+            <param name="wheel3_name">third_wheel_joint</param>
             <param name="loop_rate">30</param>
-            <param name="device">/dev/pts/6</param>
-            <param name="baudrate">115200</param>
             <param name="timeout_ms">10000</param>
             <param name="enc_counts_per_rev">1600</param>
         </hardware>
-        <joint name="roue_avant_joint">
+        <joint name="first_wheel_joint">
             <command_interface name="velocity">
                 <param name="min">-10</param>
@@ -21,5 +24,5 @@
             <state_interface name="velocity"/>
         </joint>
-        <joint name="roue_gauche_joint">
+        <joint name="second_wheel_joint">
             <command_interface name="velocity">
                 <param name="min">-10</param>
@@ -29,5 +32,5 @@
             <state_interface name="velocity"/>
         </joint>
-        <joint name="roue_arriere_joint">
+        <joint name="third_wheel_joint">
             <command_interface name="velocity">
                 <param name="min">-10</param>
