Commit message: Simulation now works in harmonic with old controller

File: robot/description/gazebo_control.xacro (robot description, xacro)
@@ -2,20 +2,14 @@
 <robot xmlns:xacro="http://www.ros.org/wiki/xacro">
     <gazebo>
-        <plugin name="ezbot_propulsion_gazebo_plugin" filename="libezbot_propulsion_gazebo_plugin.so">
+        <plugin filename="libgz_ros2_control-system.so" name="gz_ros2_control::GazeboSimROS2ControlPlugin">
+            <!--
             <North>first_wheel_joint</North>
             <West>second_wheel_joint</West>
             <South>third_wheel_joint</South>
-            <robotRadius>0.17</robotRadius>
-            <wheel_diameter>0.06</wheel_diameter>
-            <wheelDiameter>0.06</wheelDiameter>
-            <stepsPerRevolution>200</stepsPerRevolution>
-            <microstepping>16</microstepping>
-            <publish_odom>true</publish_odom>
-            <publish_odom_tf>false</publish_odom_tf>
-            <publish_wheel_tf>true</publish_wheel_tf>
-            <robotBaseFrame>base_link</robotBaseFrame>
-            <odometry_frame>odom</odometry_frame>
-            <publishOdom>true</publishOdom>
-            <publishOdomTF>true</publishOdomTF>
+            <robot_param>robot_description</robot_param>
+            <robot_param_node>robot_state_publisher</robot_param_node>
+            <parameters>$(find ezbot-v2)/config/gazebo_controller.yaml</parameters>
+            -->
+            <parameters>$(find ezbot-v2)/config/omnidirectional_controller.yaml</parameters>
         </plugin>
     </gazebo>

File: robot/description/roller/roller.urdf.xacro (robot description, xacro)
@@ -45,5 +45,5 @@
             <ode>
                 <max_vel>10</max_vel>
-                <min_depth>0.01</min_depth>
+                <min_depth>0.001</min_depth>
             </ode>
             </contact>

File: robot/description/ros2_control.xacro (robot description, xacro)
@@ -1,10 +1,8 @@
 <?xml version="1.0"?>
 <robot xmlns:xacro="http://www.ros.org/wiki/xacro">
+    <!--
     <ros2_control name="hellothere" type="system">
         <hardware>
             <plugin>omnidrive3_rppico/omnidrive3RpPicoHardware</plugin>
-            <!--
-            <param name="device">/dev/pts/6</param>
-            -->
             <param name="device">/dev/pts/69</param>
             <param name="baudrate">115200</param>
@@ -41,5 +39,4 @@
         </joint>
     </ros2_control>
-    <!--
     <ros2_control name="helloagain" type="system">
         <hardware>
@@ -60,3 +57,32 @@
     </ros2_control>
     -->
+    <ros2_control name="GazeboSimSystem" type="system">
+        <hardware>
+            <plugin>gz_ros2_control/GazeboSimSystem</plugin>
+        </hardware>
+        <joint name="first_wheel_joint">
+            <command_interface name="velocity">
+                <param name="min">-10</param>
+                <param name="max">10</param>
+            </command_interface>
+            <state_interface name="position"/>
+            <state_interface name="velocity"/>
+        </joint>
+        <joint name="second_wheel_joint">
+            <command_interface name="velocity">
+                <param name="min">-10</param>
+                <param name="max">10</param>
+            </command_interface>
+            <state_interface name="position"/>
+            <state_interface name="velocity"/>
+        </joint>
+        <joint name="third_wheel_joint">
+            <command_interface name="velocity">
+                <param name="min">-10</param>
+                <param name="max">10</param>
+            </command_interface>
+            <state_interface name="position"/>
+            <state_interface name="velocity"/>
+        </joint>
+    </ros2_control>
 </robot>
