Commit message: Refactored code to change to 3 wheeled controller
- need to change the formulas for the wheel velocities

File: robot/description/robot.urdf.xacro (robot description, xacro)
@@ -3,7 +3,7 @@
     <xacro:include filename="robot_core.xacro" />
     <xacro:include filename="gazebo_control.xacro" />
+    <xacro:include filename="ros2_control.xacro" />
     <!--
     <xacro:include filename="lidar.xacro"/>
-    <xacro:include filename="ros2_control.xacro" />
     <xacro:include filename="camera.xacro" />
     <xacro:include filename="imu.xacro" />

File: robot/description/ros2_control.xacro (robot description, xacro)
@@ -3,11 +3,10 @@
     <ros2_control name="hellothere" type="system">
         <hardware>
-            <plugin>omnidrive_rppico/OmniDriveRpPicoHardware</plugin>
-            <param name="front_wheel_name">roue_avant_joint</param>
-            <param name="left_wheel_name">roue_gauche_joint</param>
-            <param name="back_wheel_name">roue_arriere_joint</param>
-            <param name="right_wheel_name">roue_droite_joint</param>
+            <plugin>omnidrive3_rppico/omnidrive3RpPicoHardware</plugin>
+            <param name="wheel1_name">roue_avant_joint</param>
+            <param name="wheel2_name">roue_gauche_joint</param>
+            <param name="wheel3_name">roue_arriere_joint</param>
             <param name="loop_rate">30</param>
-            <param name="device">/dev/ttyAMA1</param>
+            <param name="device">/dev/pts/6</param>
             <param name="baudrate">115200</param>
             <param name="timeout_ms">10000</param>
@@ -38,14 +37,7 @@
             <state_interface name="velocity"/>
         </joint>
-        <joint name="roue_droite_joint">
-            <command_interface name="velocity">
-                <param name="min">-10</param>
-                <param name="max">10</param>
-            </command_interface>
-            <state_interface name="position"/>
-            <state_interface name="velocity"/>
-        </joint>
     </ros2_control>
-     <ros2_control name="helloagain" type="system">
+    <!--
+    <ros2_control name="helloagain" type="system">
         <hardware>
             <plugin>actuators_rppico_h_i/ActuatorsRpPicoHardware</plugin>
@@ -64,3 +56,4 @@
         </joint>
     </ros2_control>
+    -->
 </robot>

Commit message: Changed robots visuals

File: robot/description/robot.urdf.xacro (robot description, xacro)
@@ -1,11 +1,11 @@
 <?xml version="1.0"?>
 <robot xmlns:xacro="http://www.ros.org/wiki/xacro"  name="robot">
+    <xacro:arg name="namespace" default=""/>
     <xacro:include filename="robot_core.xacro" />
-    <xacro:include filename="gazebo_control.xacro" />
+    <xacro:include filename="gazebo_control.xacro"/>
     <xacro:include filename="ros2_control.xacro" />
     <xacro:include filename="camera.xacro" />
     <!--
     <xacro:include filename="lidar.xacro"/>
-    <xacro:include filename="camera.xacro" />
     <xacro:include filename="imu.xacro" />
     -->

File: robot/description/robot_core.xacro (robot description, xacro)
@@ -176,23 +176,41 @@
     <xacro:wheel_gazebo_v0 prefix="third"/>
     <link name="chassis">
-        <visual>
-            <origin xyz="0.0 0 0.0"/>
-            <geometry>
-                <mesh filename="model://ezbotv2/ezbotv2.stl" scale="0.001 0.001 0.001" />
-            </geometry>
-            <material name="gray">
-                <color rgba="0.5 0.5 0.5 1"/>
-            </material>
-        </visual>
-        <collision>
-            <origin xyz="0.0 0 0.175"/>
-            <geometry>
-                <box size="0.11 0.11 0.35"/>
-            </geometry>
-        </collision>
-        <xacro:inertial_box mass="0.5" x="0.11" y="0.11" z="0.35">
-            <origin xyz="0.0 0 0.175" rpy="0 0 0"/>
-        </xacro:inertial_box>
-    </link>
+      <visual>
+          <origin xyz="0.0 0 0.0"/>
+          <geometry>
+              <mesh filename="model://ezbotv2/ezbotv2.dae" scale="0.001 0.001 0.001" />
+          </geometry>
+          <material name="red"/>
+      </visual>
+      <collision>
+          <origin xyz="0.0 0 0.0"/>
+          <geometry>
+            <mesh filename="model://ezbotv2/ezbotv2.dae" scale="0.001 0.001 0.001" />
+          </geometry>
+      </collision>
+    </link>
+    <link name="aruco">
+      <visual>
+          <origin xyz="0.0 0 0.0"/>
+          <geometry>
+              <mesh filename="model://aruco_tags/aruco_tag_1.dae" scale="1 1 1" />
+          </geometry>
+      </visual>
+      <collision>
+          <origin xyz="0.0 0 0.0"/>
+          <geometry>
+            <mesh filename="model://aruco_tags/aruco_tag_1.dae" scale="1 1 1" />
+          </geometry>
+      </collision>
+      <xacro:inertial_box mass="0.5" x="0.11" y="0.11" z="0.35">
+          <origin xyz="0.0 0 0.0" rpy="0 0 0"/>
+      </xacro:inertial_box>
+    </link>
+    <joint name="aruco-joint" type="fixed">
+      <parent link="chassis"/>
+      <child link="aruco"/>
+      <origin xyz="0 0 0.47"/>
+    </joint>
+  <!--
     <gazebo reference="chassis">
         <visual>
@@ -205,4 +223,5 @@
         </visual>
     </gazebo>
+    -->
     <!--bloc aruco-->
     <!--

Commit message: Added World with plants and parametized aruco tags

File: robot/description/robot.urdf.xacro (robot description, xacro)
@@ -2,4 +2,5 @@
 <robot xmlns:xacro="http://www.ros.org/wiki/xacro"  name="robot">
     <xacro:arg name="namespace" default=""/>
+    <xacro:arg name="color" default="blue"/>
     <xacro:include filename="robot_core.xacro" />
     <xacro:include filename="gazebo_control.xacro"/>

File: robot/description/robot_core.xacro (robot description, xacro)
@@ -1,4 +1,6 @@
 <?xml version="1.0"?>
 <robot xmlns:xacro="http://www.ros.org/wiki/xacro" >
+    <arg name="color" default="blue"/>
+    <xacro:property name="cmp_color" value="$(arg color)"/>
     <xacro:include filename="inertial_macros.xacro" />
     <xacro:include filename="$(find ezbot-v2)/description/omni_wheel/omni_wheel.urdf.xacro" />
@@ -194,5 +196,10 @@
           <origin xyz="0.0 0 0.0"/>
           <geometry>
-              <mesh filename="model://aruco_tags/aruco_tag_1.dae" scale="1 1 1" />
+              <xacro:if value='${cmp_color == "blue"}'>
+                <mesh filename="model://aruco_tags/aruco_tag_1.dae" scale="1 1 1" />
+              </xacro:if>
+              <xacro:if value="${cmp_color == 'yellow'}">
+                <mesh filename="model://aruco_tags/aruco_tag_6.dae" scale="1 1 1" />
+              </xacro:if>
           </geometry>
       </visual>
