Commit message: Added labels to objects in the scene and 1 segmentation camera

File: robot/description/camera.xacro (robot description, xacro)
@@ -1,10 +1,16 @@
 <?xml version="1.0"?>
 <robot xmlns:xacro="http://www.ros.org/wiki/xacro" >
-    <joint name="camera_joint" type="fixed">
+    <xacro:property name="camera_downward_angle" value="0.8"/>
+    <xacro:property name="camera_horizontal_fov" value="2.0944"/>
+    <xacro:property name="camera_horizontal_pixels" value="1280"/>
+    <xacro:property name="camera_vertical_pixels" value="720"/>
+    <xacro:property name="camera_framerate" value="10"/>
+    <joint name="camera1_joint" type="fixed">
         <parent link="chassis"/>
-        <child link="camera_link"/>
-        <origin xyz="0.128 0 0.241" rpy="0 0.18 0"/>
+        <child link="camera1_link"/>
+        <origin xyz="0 -0.05 0.32" rpy="0 ${camera_downward_angle} -1.57"/>
     </joint>
-    <link name="camera_link">
+    <link name="camera1_link">
+        <origin xyz="0 0 0" rpy="0 0 -1.57"/>
         <visual>
             <geometry>
@@ -13,26 +19,87 @@
             <material name="black"/>
         </visual>
+    </link>
+    <joint name="camera1_optical_joint" type="fixed">
+        <parent link="camera1_link"/>
+        <child link="camera1_link_optical"/>
+        <origin xyz="0 0 0" rpy="${-pi/2} 0 ${-pi/2}"/>
+    </joint>
+    <link name="camera1_link_optical"></link>
+    <gazebo reference="camera1_link">
+        <material>Gazebo/Black</material>
+        <sensor name="camera1" type="camera">
+            <visualize>1</visualize>
+            <camera>
+            <horizontal_fov>${camera_horizontal_fov}</horizontal_fov> <!--120 degrees-->
+            <image>
+                <width>${camera_horizontal_pixels}</width>
+                <height>${camera_vertical_pixels}</height>
+            </image>
+            <clip>
+                <near>0.1</near>
+                <far>100</far>
+            </clip>
+            <!--
+            <distortion>
+                <k2>-5.784303605943902360e-01</k2>
+                <k3>-8.740723680089258069e-03</k3>
+                <p1>1.359451618091441112e-03</p1>
+                <p2>1.640043376158566713e-01</p2>
+                <center>0.5 0.5</center>
+            </distortion>
+            <lens>
+                <type>pinhole</type>
+                <scale_to_hfov>false</scale_to_hfov>
+                <intrinsics>
+                <fx>4.970870507466349295e+02</fx>
+                <fy>4.976011127668800782e+02</fy>
+                <cx>3.168387473166100108e+02</cx>
+                <cy>2.342740555042151982e+02</cy>
+                <s>0.0</s>
+                </intrinsics>
+            </lens>
+            -->
+            </camera>
+            <always_on>1</always_on>
+            <update_rate>${camera_framerate}</update_rate>
+            <topic>$(arg namespace)/camera1</topic>
+        </sensor>
+    </gazebo>
+    <joint name="camera2_base_joint" type="fixed">
+        <parent link="chassis"/>
+        <child link="camera2_base_rotated"/>
+        <origin xyz="0 0 0" rpy="0 0 ${2*pi/3}"/>
+    </joint>
+    <link name="camera2_base_rotated">
+    </link>
+    <joint name="camera2_joint" type="fixed">
+        <parent link="camera2_base_rotated"/>
+        <child link="camera2_link"/>
+        <origin xyz="0 -0.05 0.32" rpy="0 ${camera_downward_angle} -1.57"/>
+    </joint>
+    <link name="camera2_link">
+        <origin xyz="0 0 0" rpy="0 0 -1.57"/>
         <visual>
-            <origin xyz="0 0 -0.05"/>
             <geometry>
-                <cylinder radius="0.002" length="0.1"/>
+                <box size="0.010 0.03 0.03"/>
             </geometry>
             <material name="black"/>
         </visual>
     </link>
-    <joint name="camera_optical_joint" type="fixed">
-        <parent link="camera_link"/>
-        <child link="camera_link_optical"/>
+    <joint name="camera2_optical_joint" type="fixed">
+        <parent link="camera2_link"/>
+        <child link="camera2_link_optical"/>
         <origin xyz="0 0 0" rpy="${-pi/2} 0 ${-pi/2}"/>
     </joint>
-    <link name="camera_link_optical"></link>
-    <gazebo reference="camera_link">
+    <link name="camera2_link_optical"></link>
+    <gazebo reference="camera2_link">
         <material>Gazebo/Black</material>
-        <sensor name="camera" type="camera">
+        <sensor name="camera2" type="camera">
+            <visualize>1</visualize>
             <camera>
-            <horizontal_fov>1.047</horizontal_fov>
+            <horizontal_fov>${camera_horizontal_fov}</horizontal_fov> <!--120 degrees-->
             <image>
-                <width>1000</width>
-                <height>1000</height>
+                <width>${camera_horizontal_pixels}</width>
+                <height>${camera_vertical_pixels}</height>
             </image>
             <clip>
@@ -42,7 +109,70 @@
             </camera>
             <always_on>1</always_on>
-            <update_rate>10</update_rate>
-            <visualize>true</visualize>
-            <topic>$(arg namespace)/camera</topic>
+            <update_rate>${camera_framerate}</update_rate>
+            <topic>$(arg namespace)/camera2</topic>
+        </sensor>
+    </gazebo>
+    <joint name="camera3_base_joint" type="fixed">
+        <parent link="chassis"/>
+        <child link="camera3_base_rotated"/>
+        <origin xyz="0 0 0" rpy="0 0 ${-2*pi/3}"/>
+    </joint>
+    <link name="camera3_base_rotated">
+    </link>
+    <joint name="camera3_joint" type="fixed">
+        <parent link="camera3_base_rotated"/>
+        <child link="camera3_link"/>
+        <origin xyz="0 -0.05 0.32" rpy="0 ${camera_downward_angle} -1.57"/>
+    </joint>
+    <link name="camera3_link">
+        <origin xyz="0 0 0" rpy="0 0 -1.57"/>
+        <visual>
+            <geometry>
+                <box size="0.010 0.03 0.03"/>
+            </geometry>
+            <material name="black"/>
+        </visual>
+    </link>
+    <joint name="camera3_optical_joint" type="fixed">
+        <parent link="camera3_link"/>
+        <child link="camera3_link_optical"/>
+        <origin xyz="0 0 0" rpy="${-pi/2} 0 ${-pi/2}"/>
+    </joint>
+    <link name="camera3_link_optical"></link>
+    <gazebo reference="camera3_link">
+        <sensor name="camera3" type="camera">
+            <visualize>1</visualize>
+            <camera>
+            <horizontal_fov>${camera_horizontal_fov}</horizontal_fov>
+            <image>
+                <width>${camera_horizontal_pixels}</width>
+                <height>${camera_vertical_pixels}</height>
+            </image>
+            <clip>
+                <near>0.1</near>
+                <far>100</far>
+            </clip>
+            </camera>
+            <always_on>1</always_on>
+            <update_rate>${camera_framerate}</update_rate>
+            <topic>$(arg namespace)/camera3</topic>
+        </sensor>
+        <sensor name="segmentation_camera" type="segmentation">
+        <topic>$(arg namespace)/camera3</topic>
+        <camera>
+            <segmentation_type>instance</segmentation_type>
+            <horizontal_fov>${camera_horizontal_fov}</horizontal_fov>
+            <image>
+                <width>${camera_horizontal_pixels}</width>
+                <height>${camera_vertical_pixels}</height>
+            </image>
+            <clip>
+            <near>0.1</near>
+            <far>100</far>
+            </clip>
+        </camera>
+        <always_on>1</always_on>
+        <update_rate>${camera_framerate}</update_rate>
+        <visualize>true</visualize>
         </sensor>
     </gazebo>
