Commit message: Added back 2D LIDAR

File: robot/description/lidar.xacro (robot description, xacro)
@@ -4,5 +4,5 @@
         <parent link="chassis"/>
         <child link="base_laser"/>
-        <origin xyz="0.055 0 0.41" rpy="0 0 0"/>
+        <origin xyz="0.0 0 0.41" rpy="0 0 0"/>
     </joint>
     <joint name="ldlidar_node" type="fixed">
@@ -45,6 +45,10 @@
     <gazebo reference="base_laser">
         <material>Gazebo/Black</material>
-        <sensor name="laser" type="ray">
-            <pose> 0.055 0 0.03 0 0 0 </pose>
+        <sensor name="gpu_lidar" type="gpu_lidar">
+            <pose> 0 0 0 0 0 0 </pose>
+            <topic>$(arg namespace)/lidar</topic>
+            <!--
+            <gz_frame_id>$(arg namespace)/base_laser</gz_frame_id>
+            -->
             <visualize>true</visualize>
             <update_rate>10</update_rate>
@@ -62,11 +66,4 @@
                 </range>
             </ray>
-            <plugin name="laser_controller" filename="libgazebo_ros_ray_sensor.so">
-                <ros>
-                    <argument>~/out:=lidar/ldlidar_node/scan</argument>
-                </ros>
-                <output_type>sensor_msgs/LaserScan</output_type>
-                <frame_name>base_laser</frame_name>
-            </plugin>
         </sensor>
     </gazebo>

File: robot/description/robot.urdf.xacro (robot description, xacro)
@@ -7,6 +7,6 @@
     <xacro:include filename="ros2_control.xacro" />
     <xacro:include filename="camera.xacro" />
+    <xacro:include filename="lidar.xacro"/>
     <!--
-    <xacro:include filename="lidar.xacro"/>
     <xacro:include filename="imu.xacro" />
     -->
