Commit message: changed how mesh files are declare for rviz2 to find them

File: src/ezbot-v2/description/omni_wheel/omni_wheel.urdf.xacro (robot description, xacro)
@@ -14,10 +14,10 @@
 	  <visual>
 		<geometry>
-		  <mesh filename="$(find ezbot-v2)/meshes/DAE/omni_wheel/omni_wheel.dae"/>
+		  <mesh filename="file://$(find ezbot-v2)/meshes/DAE/omni_wheel/omni_wheel.dae"/>
 		</geometry>
 	  </visual>
 	  <collision>
 		<geometry>
-		  <mesh filename="$(find ezbot-v2)/meshes/STL/omni_wheel/omni_wheel.stl"/>
+		  <mesh filename="file://$(find ezbot-v2)/meshes/STL/omni_wheel/omni_wheel.stl"/>
 		</geometry>
 	  </collision>

File: src/ezbot-v2/description/robot.urdf.xacro (robot description, xacro)
@@ -8,6 +8,4 @@
     <xacro:include filename="camera.xacro" />
     <xacro:include filename="lidar.xacro"/>
-    <!--
     <xacro:include filename="imu.xacro" />
-    -->
 </robot>

File: src/ezbot-v2/description/robot_core.xacro (robot description, xacro)
@@ -37,6 +37,7 @@
     </joint>
     <xacro:property name="M_PI" value="3.14159274"/>
+    <xacro:property name="wheel_distance" value="0.175"/>
     <xacro:wheel_v0 prefix="first" parent="base_link">
-        <origin xyz="0.0 0.175 0.03" rpy="0 0 0"/>
+        <origin xyz="${wheel_distance} 0.0 0.03" rpy="0 0 ${-M_PI/2}"/>
         <axis xyz="0 1 0"/>
     </xacro:wheel_v0>
@@ -83,5 +84,8 @@
     <!-- 2nd wheel -->
   <xacro:wheel_v0 prefix="second" parent="base_link">
-	<origin xyz="-0.1515 -0.0875 0.03" rpy="0 0 ${2*M_PI/3}"/>
+  <!--
+	<origin xyz="-0.0875 0.1515 0.03" rpy="0 0 ${M_PI/6}"/>
+  -->
+	<origin xyz="${-0.5*wheel_distance} ${wheel_distance* 0.8660254038335881} 0.03" rpy="0 0 ${M_PI/6}"/>
 	<axis xyz="0 1 0"/>
   </xacro:wheel_v0>
@@ -128,5 +132,5 @@
 <!-- 3rd wheel -->
   <xacro:wheel_v0 prefix="third" parent="base_link">
-	<origin xyz="0.1515 -0.0875 0.03" rpy="0 0 ${-2*M_PI/3}"/>
+	<origin xyz="${-0.5*wheel_distance} ${-wheel_distance* 0.8660254038335881} 0.03" rpy="0 0 ${2*M_PI/3 +M_PI/6}"/>
 	<axis xyz="0 1 0"/>
   </xacro:wheel_v0>
@@ -179,16 +183,21 @@
     <link name="chassis">
       <visual>
-          <origin xyz="0.0 0 0.0"/>
-          <geometry>
-              <mesh filename="model://ezbotv2/ezbotv2.dae" scale="0.001 0.001 0.001" />
+          <origin xyz="0 0 0" rpy="0 0 ${-M_PI/2}"/>
+          <geometry>
+              <mesh filename="file://$(find ezbot-v2)/models/ezbotv2/ezbotv2.dae" scale="0.001 0.001 0.001" />
           </geometry>
           <material name="red"/>
       </visual>
       <collision>
-          <origin xyz="0.0 0 0.0"/>
-          <geometry>
-            <mesh filename="model://ezbotv2/ezbotv2.dae" scale="0.001 0.001 0.001" />
+          <origin xyz="0 0 0" rpy="0 0 ${-M_PI/2}"/>
+          <geometry>
+            <mesh filename="file://$(find ezbot-v2)/models/ezbotv2/ezbotv2.dae" scale="0.001 0.001 0.001" />
           </geometry>
       </collision>
+      <inertial>
+          <origin xyz="0 0 0" rpy="0 0 0"/>
+          <mass value="3.0"/>
+          <inertia ixx="0.0001" ixy="0" ixz="0" iyy="0.0001" iyz="0" izz="0.0001"/>
+      </inertial>
     </link>
     <link name="aruco">
@@ -197,8 +206,8 @@
           <geometry>
               <xacro:if value='${cmp_color == "blue"}'>
-                <mesh filename="model://aruco_tags/aruco_tag_1.dae" scale="1 1 1" />
+                <mesh filename="file://$(find ezbot-v2)/models/aruco_tags/aruco_tag_1.dae" scale="1 1 1" />
               </xacro:if>
               <xacro:if value="${cmp_color == 'yellow'}">
-                <mesh filename="model://aruco_tags/aruco_tag_6.dae" scale="1 1 1" />
+                <mesh filename="file://$(find ezbot-v2)/models/aruco_tags/aruco_tag_6.dae" scale="1 1 1" />
               </xacro:if>
           </geometry>
@@ -207,5 +216,5 @@
           <origin xyz="0.0 0 0.0"/>
           <geometry>
-            <mesh filename="model://aruco_tags/aruco_tag_1.dae" scale="1 1 1" />
+            <mesh filename="file://$(find ezbot-v2)/models/aruco_tags/aruco_tag_1.dae" scale="1 1 1" />
           </geometry>
       </collision>

File: src/ezbot-v2/description/roller/roller.urdf.xacro (robot description, xacro)
@@ -17,10 +17,10 @@
     <visual>
       <geometry>
-        <mesh filename="$(find ezbot-v2)/meshes/DAE/roller/roller.dae"/>
+        <mesh filename="file://$(find ezbot-v2)/meshes/DAE/roller/roller.dae"/>
       </geometry>
 	  </visual>
     <collision>
       <geometry>
-        <mesh filename="$(find ezbot-v2)/meshes/STL/roller/roller.stl"/>
+        <mesh filename="file://$(find ezbot-v2)/meshes/STL/roller/roller.stl"/>
       </geometry>
 	  </collision>
