Commit message: Overhauled poteau positing system, now works pretty well Need to fix for genneric LIDAR orientation

File: src/ezbot-v2/description/lidar.xacro (robot description, xacro)
@@ -4,5 +4,5 @@
         <parent link="chassis"/>
         <child link="base_laser"/>
-        <origin xyz="0.0 0 0.41" rpy="0 0 1.0471975512"/>
+        <origin xyz="0.0 0 0.41" rpy="0 0 0"/>
     </joint>
     <joint name="ldlidar_node" type="fixed">
