Commit message: added working IMU, LIDAR, and cameras

File: src/ezbot-v2/description/camera.xacro (robot description, xacro)
@@ -9,5 +9,5 @@
         <parent link="chassis"/>
         <child link="camera1_link"/>
-        <origin xyz="0 -0.05 0.32" rpy="0 ${camera_downward_angle} -1.57"/>
+        <origin xyz="-0.05 0 0.32" rpy="0 ${camera_downward_angle} -3.141592"/>
     </joint>
     <link name="camera1_link">
@@ -69,5 +69,5 @@
         <parent link="chassis"/>
         <child link="camera2_base_rotated"/>
-        <origin xyz="0 0 0" rpy="0 0 ${2*pi/3}"/>
+        <origin xyz="0 0 0" rpy="0 0 ${pi/6}"/>
     </joint>
     <link name="camera2_base_rotated">
@@ -116,5 +116,5 @@
         <parent link="chassis"/>
         <child link="camera3_base_rotated"/>
-        <origin xyz="0 0 0" rpy="0 0 ${-2*pi/3}"/>
+        <origin xyz="0 0 0" rpy="0 0 ${-7*pi/6}"/>
     </joint>
     <link name="camera3_base_rotated">

File: src/ezbot-v2/description/imu.xacro (robot description, xacro)
@@ -15,77 +15,22 @@
     </link>
     <gazebo reference="imu">
-        <material>Gazebo/Black</material>
-        <gravity>true</gravity>
-        <sensor name="imu_sensor" type="imu">
-            <always_on>true</always_on>
-            <update_rate>100</update_rate>
-            <visualize>true</visualize>
-            <topic>__default_topic__</topic>
-            <plugin filename="libgazebo_ros_imu_sensor.so" name="imu_plugin">
-                <topicName>imu</topicName>
-                <bodyName>imu</bodyName>
-                <updateRateHZ>10.0</updateRateHZ>
-                <gaussianNoise>0.0</gaussianNoise>
-                <xyzOffset>0 0 0</xyzOffset>
-                <rpyOffset>0 0 0</rpyOffset>
-                <frameName>imu</frameName>
-                <initialOrientationAsReference>false</initialOrientationAsReference>
-            </plugin>
-            <pose>0 0 0 0 0 0</pose>
-            <imu>
-            <angular_velocity>
+      <sensor name="imu_sensor" type="imu">
+        <always_on>1</always_on>
+        <update_rate>10</update_rate>
+        <visualize>true</visualize>
+        <topic>$(arg namespace)/imu</topic>
+        <gz_frame_id>$(arg namespace)/imu</gz_frame_id>
+        <!-- cf http://sdformat.org/spec?ver=1.10&elem=sensor#sensor_imu -->
+        <imu>
+          <angular_velocity>
             <x>
               <noise type="gaussian">
-                <mean>0.0</mean>
-                <stddev>2e-4</stddev>
-                <bias_mean>0.0000075</bias_mean>
-                <bias_stddev>0.0000008</bias_stddev>
+                <mean>0</mean>
+                <stddev>0.01</stddev>
               </noise>
             </x>
-            <y>
-              <noise type="gaussian">
-                <mean>0.0</mean>
-                <stddev>2e-4</stddev>
-                <bias_mean>0.0000075</bias_mean>
-                <bias_stddev>0.0000008</bias_stddev>
-              </noise>
-            </y>
-            <z>
-              <noise type="gaussian">
-                <mean>0.0</mean>
-                <stddev>2e-4</stddev>
-                <bias_mean>0.0000075</bias_mean>
-                <bias_stddev>0.0000008</bias_stddev>
-              </noise>
-            </z>
-            </angular_velocity>
-            <linear_acceleration>
-            <x>
-              <noise type="gaussian">
-                <mean>0.0</mean>
-                <stddev>1.7e-2</stddev>
-                <bias_mean>0.1</bias_mean>
-                <bias_stddev>0.001</bias_stddev>
-              </noise>
-            </x>
-            <y>
-              <noise type="gaussian">
-                <mean>0.0</mean>
-                <stddev>1.7e-2</stddev>
-                <bias_mean>0.1</bias_mean>
-                <bias_stddev>0.001</bias_stddev>
-              </noise>
-            </y>
-            <z>
-              <noise type="gaussian">
-                <mean>0.0</mean>
-                <stddev>1.7e-2</stddev>
-                <bias_mean>0.1</bias_mean>
-                <bias_stddev>0.001</bias_stddev>
-              </noise>
-            </z>
-            </linear_acceleration>
-            </imu>
-        </sensor>
+          </angular_velocity>
+        </imu>
+      </sensor>
     </gazebo>
 </robot>

File: src/ezbot-v2/description/lidar.xacro (robot description, xacro)
@@ -4,5 +4,5 @@
         <parent link="chassis"/>
         <child link="base_laser"/>
-        <origin xyz="0.0 0 0.41" rpy="0 0 0"/>
+        <origin xyz="0.0 0 0.41" rpy="0 0 1.0471975512"/>
     </joint>
     <joint name="ldlidar_node" type="fixed">
@@ -23,5 +23,5 @@
         <visual>
             <geometry>
-                <cylinder radius="0.02" length="0.04"/>
+                <cylinder radius="0.05" length="0.04"/>
             </geometry>
             <material name="black"/>
@@ -30,5 +30,5 @@
             <origin xyz="0 0 -0.05"/>
             <geometry>
-                <cylinder radius="0.01" length="0.1"/>
+                <cylinder radius="0.05" length="0.1"/>
             </geometry>
             <material name="black"/>
@@ -36,5 +36,5 @@
         <collision>
             <geometry>
-                <cylinder radius="0.02" length="0.04"/>
+                <cylinder radius="0.05" length="0.04"/>
             </geometry>
         </collision>
@@ -43,4 +43,5 @@
         </xacro:inertial_cylinder>
     </link>
+    <xacro:property name="noise" value="0.01"/>
     <gazebo reference="base_laser">
         <material>Gazebo/Black</material>
@@ -48,7 +49,5 @@
             <pose> 0 0 0 0 0 0 </pose>
             <topic>$(arg namespace)/lidar</topic>
-            <!--
             <gz_frame_id>$(arg namespace)/base_laser</gz_frame_id>
-            -->
             <visualize>true</visualize>
             <update_rate>10</update_rate>
@@ -65,5 +64,15 @@
                     <max>12</max>
                 </range>
+                <noise>
+                    <type>gaussian</type>
+                    <mean>0.01</mean>
+                    <stddev>0.01</stddev>
+                </noise>
             </ray>
+            <!-- Noise
+            <plugin name="gazebo_ros_laser_controller" filename="libgazebo_ros_lidar_gpu.so">
+                <gaussianNoise>${noise}</gaussianNoise>
+            </plugin>
+            -->
         </sensor>
     </gazebo>

Commit message: Adding new world and fixed robot description

File: src/ezbot-v2/description/camera.xacro (robot description, xacro)
@@ -2,5 +2,5 @@
 <robot xmlns:xacro="http://www.ros.org/wiki/xacro" >
     <xacro:property name="camera_downward_angle" value="0.8"/>
-    <xacro:property name="camera_horizontal_fov" value="2.0944"/>
+    <xacro:property name="camera_horizontal_fov" value="1.8906"/> <!--108 degrees-->
     <xacro:property name="camera_horizontal_pixels" value="1280"/>
     <xacro:property name="camera_vertical_pixels" value="720"/>
@@ -15,7 +15,7 @@
         <visual>
             <geometry>
-                <box size="0.010 0.03 0.03"/>
+                <box size="0.010 0.04 0.04"/>
             </geometry>
-            <material name="black"/>
+            <material name="grey"/>
         </visual>
     </link>
@@ -27,6 +27,7 @@
     <link name="camera1_link_optical"></link>
     <gazebo reference="camera1_link">
-        <material>Gazebo/Black</material>
+        <material>Gazebo/Grey</material>
         <sensor name="camera1" type="camera">
+            <topic>$(arg namespace)/camera1/img_raw</topic>
             <visualize>1</visualize>
             <camera>
@@ -63,5 +64,4 @@
             <always_on>1</always_on>
             <update_rate>${camera_framerate}</update_rate>
-            <topic>$(arg namespace)/camera1</topic>
         </sensor>
     </gazebo>
@@ -82,7 +82,7 @@
         <visual>
             <geometry>
-                <box size="0.010 0.03 0.03"/>
+                <box size="0.010 0.04 0.04"/>
             </geometry>
-            <material name="black"/>
+            <material name="grey"/>
         </visual>
     </link>
@@ -94,5 +94,5 @@
     <link name="camera2_link_optical"></link>
     <gazebo reference="camera2_link">
-        <material>Gazebo/Black</material>
+        <material>Gazebo/Grey</material>
         <sensor name="camera2" type="camera">
             <visualize>1</visualize>
@@ -110,5 +110,5 @@
             <always_on>1</always_on>
             <update_rate>${camera_framerate}</update_rate>
-            <topic>$(arg namespace)/camera2</topic>
+            <topic>$(arg namespace)/camera2/img_raw</topic>
         </sensor>
     </gazebo>
@@ -129,7 +129,7 @@
         <visual>
             <geometry>
-                <box size="0.010 0.03 0.03"/>
+                <box size="0.010 0.04 0.04"/>
             </geometry>
-            <material name="black"/>
+            <material name="grey"/>
         </visual>
     </link>
@@ -141,4 +141,5 @@
     <link name="camera3_link_optical"></link>
     <gazebo reference="camera3_link">
+        <material>Gazebo/Grey</material>
         <sensor name="camera3" type="camera">
             <visualize>1</visualize>
@@ -156,8 +157,8 @@
             <always_on>1</always_on>
             <update_rate>${camera_framerate}</update_rate>
-            <topic>$(arg namespace)/camera3</topic>
+            <topic>$(arg namespace)/camera3/img_raw</topic>
         </sensor>
         <sensor name="segmentation_camera" type="segmentation">
-        <topic>$(arg namespace)/camera3</topic>
+        <topic>$(arg namespace)/camera3_segm</topic>
         <camera>
             <segmentation_type>instance</segmentation_type>

File: src/ezbot-v2/description/lidar.xacro (robot description, xacro)
@@ -23,5 +23,5 @@
         <visual>
             <geometry>
-                <cylinder radius="0.05" length="0.04"/>
+                <cylinder radius="0.04" length="0.04"/>
             </geometry>
             <material name="black"/>
@@ -30,5 +30,5 @@
             <origin xyz="0 0 -0.05"/>
             <geometry>
-                <cylinder radius="0.05" length="0.1"/>
+                <cylinder radius="0.04" length="0.1"/>
             </geometry>
             <material name="black"/>
@@ -36,8 +36,8 @@
         <collision>
             <geometry>
-                <cylinder radius="0.05" length="0.04"/>
+                <cylinder radius="0.04" length="0.04"/>
             </geometry>
         </collision>
-        <xacro:inertial_cylinder mass="0.1" length="0.04" radius="0.05">
+        <xacro:inertial_cylinder mass="0.1" length="0.04" radius="0.04">
             <origin xyz="0 0 0" rpy="0 0 0"/>
         </xacro:inertial_cylinder>

Commit message: working simulation with rand spawn points

File: src/ezbot-v2/description/camera.xacro (robot description, xacro)
@@ -17,5 +17,4 @@
                 <box size="0.010 0.04 0.04"/>
             </geometry>
-            <material name="grey"/>
         </visual>
     </link>
@@ -84,5 +83,4 @@
                 <box size="0.010 0.04 0.04"/>
             </geometry>
-            <material name="grey"/>
         </visual>
     </link>
@@ -131,5 +129,4 @@
                 <box size="0.010 0.04 0.04"/>
             </geometry>
-            <material name="grey"/>
         </visual>
     </link>

Commit message: Changed various description values

File: src/ezbot-v2/description/camera.xacro (robot description, xacro)
@@ -38,5 +38,5 @@
             <clip>
                 <near>0.1</near>
-                <far>100</far>
+                <far>10</far>
             </clip>
             <!--
@@ -103,5 +103,5 @@
             <clip>
                 <near>0.1</near>
-                <far>100</far>
+                <far>10</far>
             </clip>
             </camera>
@@ -156,4 +156,5 @@
             <topic>$(arg namespace)/camera3/img_raw</topic>
         </sensor>
+        <!--
         <sensor name="segmentation_camera" type="segmentation">
         <topic>$(arg namespace)/camera3_segm</topic>
@@ -167,5 +168,5 @@
             <clip>
             <near>0.1</near>
-            <far>100</far>
+            <far>10</far>
             </clip>
         </camera>
@@ -174,4 +175,5 @@
         <visualize>true</visualize>
         </sensor>
+        -->
     </gazebo>
 </robot>

File: src/ezbot-v2/description/imu.xacro (robot description, xacro)
@@ -2,5 +2,5 @@
 <robot xmlns:xacro="http://www.ros.org/wiki/xacro" >
     <joint name="imu_joint" type="fixed">
-        <parent link="chassis"/>
+        <parent link="base_link"/>
         <child link="imu"/>
         <origin xyz="0.055 0 0.175" rpy="0 0 0"/>

File: src/ezbot-v2/description/lidar.xacro (robot description, xacro)
@@ -66,6 +66,6 @@
                 <noise>
                     <type>gaussian</type>
-                    <mean>0.01</mean>
-                    <stddev>0.01</stddev>
+                    <mean>0.001</mean>
+                    <stddev>0.001</stddev>
                 </noise>
             </ray>

File: src/ezbot-v2/description/robot_core.xacro (robot description, xacro)
@@ -190,7 +190,10 @@
       </visual>
       <collision>
-          <origin xyz="0 0 0" rpy="0 0 ${-M_PI/2}"/>
-          <geometry>
+          <origin xyz="0 0 0.16" rpy="0 0 ${-M_PI/2}"/>
+           <geometry>
+              <box size="0.2 0.2 0.3"/>
+          <!--
             <mesh filename="file://$(find ezbot-v2)/models/ezbotv2/ezbotv2.dae" scale="0.001 0.001 0.001" />
+          -->
           </geometry>
       </collision>

File: src/ezbot-v2/description/roller/roller.urdf.xacro (robot description, xacro)
@@ -12,5 +12,5 @@
       Setting friction too high (1.0 tested) result in weird movement and behavior
     -->
-    <dynamics damping="0.0" friction="0.01"/>
+    <dynamics damping="0.5" friction="0.01"/>
 	</joint>
 	<link name="${prefix}_roller_link">

Commit message: Added segmentation to all camera and made it toggleable

File: src/ezbot-v2/description/camera.xacro (robot description, xacro)
@@ -6,4 +6,5 @@
     <xacro:property name="camera_vertical_pixels" value="720"/>
     <xacro:property name="camera_framerate" value="10"/>
+    <xacro:property name="camera_segm_enable" value="false"/>
     <joint name="camera1_joint" type="fixed">
         <parent link="chassis"/>
@@ -64,4 +65,24 @@
             <update_rate>${camera_framerate}</update_rate>
         </sensor>
+        <xacro:if value="${camera_segm_enable}">
+            <sensor name="segmentation_camera1" type="segmentation">
+            <topic>$(arg namespace)/camera1_segm</topic>
+            <camera>
+                <segmentation_type>instance</segmentation_type>
+                <horizontal_fov>${camera_horizontal_fov}</horizontal_fov>
+                <image>
+                    <width>${camera_horizontal_pixels}</width>
+                    <height>${camera_vertical_pixels}</height>
+                </image>
+                <clip>
+                <near>0.1</near>
+                <far>10</far>
+                </clip>
+            </camera>
+            <always_on>1</always_on>
+            <update_rate>${camera_framerate}</update_rate>
+            <visualize>true</visualize>
+            </sensor>
+        </xacro:if>
     </gazebo>
     <joint name="camera2_base_joint" type="fixed">
@@ -110,4 +131,24 @@
             <topic>$(arg namespace)/camera2/img_raw</topic>
         </sensor>
+        <xacro:if value="${camera_segm_enable}">
+            <sensor name="segmentation_camera2" type="segmentation">
+            <topic>$(arg namespace)/camera2_segm</topic>
+            <camera>
+                <segmentation_type>instance</segmentation_type>
+                <horizontal_fov>${camera_horizontal_fov}</horizontal_fov>
+                <image>
+                    <width>${camera_horizontal_pixels}</width>
+                    <height>${camera_vertical_pixels}</height>
+                </image>
+                <clip>
+                <near>0.1</near>
+                <far>10</far>
+                </clip>
+            </camera>
+            <always_on>1</always_on>
+            <update_rate>${camera_framerate}</update_rate>
+            <visualize>true</visualize>
+            </sensor>
+        </xacro:if>
     </gazebo>
     <joint name="camera3_base_joint" type="fixed">
@@ -156,24 +197,24 @@
             <topic>$(arg namespace)/camera3/img_raw</topic>
         </sensor>
-        <!--
-        <sensor name="segmentation_camera" type="segmentation">
-        <topic>$(arg namespace)/camera3_segm</topic>
-        <camera>
-            <segmentation_type>instance</segmentation_type>
-            <horizontal_fov>${camera_horizontal_fov}</horizontal_fov>
-            <image>
-                <width>${camera_horizontal_pixels}</width>
-                <height>${camera_vertical_pixels}</height>
-            </image>
-            <clip>
-            <near>0.1</near>
-            <far>10</far>
-            </clip>
-        </camera>
-        <always_on>1</always_on>
-        <update_rate>${camera_framerate}</update_rate>
-        <visualize>true</visualize>
-        </sensor>
-        -->
+        <xacro:if value="${camera_segm_enable}">
+            <sensor name="segmentation_camera3" type="segmentation">
+            <topic>$(arg namespace)/camera3_segm</topic>
+            <camera>
+                <segmentation_type>instance</segmentation_type>
+                <horizontal_fov>${camera_horizontal_fov}</horizontal_fov>
+                <image>
+                    <width>${camera_horizontal_pixels}</width>
+                    <height>${camera_vertical_pixels}</height>
+                </image>
+                <clip>
+                <near>0.1</near>
+                <far>10</far>
+                </clip>
+            </camera>
+            <always_on>1</always_on>
+            <update_rate>${camera_framerate}</update_rate>
+            <visualize>true</visualize>
+            </sensor>
+        </xacro:if>
     </gazebo>
 </robot>

Commit message: WIP, commit to edit

File: src/ezbot-v2/description/camera.xacro (robot description, xacro)
@@ -5,5 +5,5 @@
     <xacro:property name="camera_horizontal_pixels" value="1280"/>
     <xacro:property name="camera_vertical_pixels" value="720"/>
-    <xacro:property name="camera_framerate" value="10"/>
+    <xacro:property name="camera_framerate" value="5"/>
     <xacro:property name="camera_segm_enable" value="false"/>
     <joint name="camera1_joint" type="fixed">

File: src/ezbot-v2/description/lidar.xacro (robot description, xacro)
@@ -70,9 +70,4 @@
                 </noise>
             </ray>
-            <!-- Noise
-            <plugin name="gazebo_ros_laser_controller" filename="libgazebo_ros_lidar_gpu.so">
-                <gaussianNoise>${noise}</gaussianNoise>
-            </plugin>
-            -->
         </sensor>
     </gazebo>

Commit message: WIP on laptop, whatever that work was

File: src/ezbot-v2/description/camera.xacro (robot description, xacro)
@@ -3,7 +3,7 @@
     <xacro:property name="camera_downward_angle" value="0.8"/>
     <xacro:property name="camera_horizontal_fov" value="1.8906"/> <!--108 degrees-->
-    <xacro:property name="camera_horizontal_pixels" value="1280"/>
-    <xacro:property name="camera_vertical_pixels" value="720"/>
-    <xacro:property name="camera_framerate" value="10"/>
+    <xacro:property name="camera_horizontal_pixels" value="720"/>
+    <xacro:property name="camera_vertical_pixels" value="480"/>
+    <xacro:property name="camera_framerate" value="30"/>
     <xacro:property name="camera_segm_enable" value="false"/>
     <joint name="camera1_joint" type="fixed">

File: src/ezbot-v2/description/robot_core.xacro (robot description, xacro)
@@ -185,5 +185,5 @@
           <origin xyz="0 0 0" rpy="0 0 ${-M_PI/2}"/>
           <geometry>
-              <mesh filename="file://$(find ezbot-v2)/models/ezbotv2/ezbotv2.dae" scale="0.001 0.001 0.001" />
+              <mesh filename="file://$(find ezbot-v2)/models/ezbotv2/ezbotv1_5.dae" scale="1.0 1.0 1.0" />
           </geometry>
           <material name="red"/>
