Commit message: Remote calc launch file added for 2026, and changed config for wider converage

File: src/remote-calc/description/single_camera.xacro (robot description, xacro)
@@ -2,7 +2,7 @@
 <robot xmlns:xacro="http://www.ros.org/wiki/xacro" >
     <xacro:property name="camera_downward_angle" value="1.0472"/>
-    <xacro:property name="camera_horizontal_fov" value="1.8906"/> <!--108 degrees-->
-    <xacro:property name="camera_horizontal_pixels" value="1280"/>
-    <xacro:property name="camera_vertical_pixels" value="720"/>
+    <xacro:property name="camera_horizontal_fov" value="1.74533"/> <!--100 degrees-->
+    <xacro:property name="camera_horizontal_pixels" value="1920"/>
+    <xacro:property name="camera_vertical_pixels" value="1080"/>
     <xacro:property name="camera_framerate" value="10"/>
     <xacro:property name="camera_segm_enable" value="false"/>
@@ -35,5 +35,5 @@
         <parent link="remote_calc_base"/>
         <child link="camera1_link"/>
-        <origin xyz="0.0 0 0.32" rpy="0 ${camera_downward_angle} -3.141592"/>
+        <origin xyz="0.0 0 0.05" rpy="0 ${camera_downward_angle} -3.141592"/>
     </joint>
     <link name="camera1_link">
